File: VMFB-MC.kicad_sch (KiCad schematic)
At the start: 47 parts, among them J1 DISPENSE, J10 Conn_01x05_Pin, J2 EMPTY, J3 DISPENSE, J4 MOTOR, J5 PIR, J6 Conn_01x04_Pin, J7 EMPTY, J8 DEPOSIT, J9 DISPENSE, Q1 Q_Photo_NPN, Q2 Q_Photo_NPN, Q3 Q_Photo_NPN, Q4 Q_Photo_NPN, Q5 Q_Photo_NPN, Q6 Q_Photo_NPN, Q7 TIP120, Q8 TIP120, Q9 Q_Photo_NPN, U1 LM393

Commit message: MT bleeder resistor
Added bleeder resistor to the MT sensor.
Parts:
- added R18: 10K, Resistor_THT:R_Axial_DIN0207_L6.3mm_D2.5mm_P2.54mm_Vertical, symbol Device:R
Connections:
- net GND: now also R18.2
- net at J7.4 (Pin_4), R17.2: now also R18.1
Other:
- moved on the sheet: J7, R17
Changed lines of the file:
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@@
   (junction (at 217.17 152.4) (diameter 0) (color 0 0 0 0)
   )
+  (junction (at 135.89 96.52) (diameter 0) (color 0 0 0 0)
+  )
   (junction (at 201.93 142.24) (diameter 0) (color 0 0 0 0)
   )
@@
     (stroke (width 0) (type default))
   )
-  (wire (pts (xy 135.89 96.52) (xy 142.24 96.52))
+  (wire (pts (xy 135.89 91.44) (xy 142.24 91.44))
     (stroke (width 0) (type default))
   )
@@
     (stroke (width 0) (type default))
   )
-  (wire (pts (xy 135.89 99.06) (xy 142.24 99.06))
+  (wire (pts (xy 135.89 93.98) (xy 142.24 93.98))
     (stroke (width 0) (type default))
   )
@@
     (stroke (width 0) (type default))
   )
+  (wire (pts (xy 135.89 96.52) (xy 135.89 101.6))
+    (stroke (width 0) (type default))
+  )
   (wire (pts (xy 217.17 152.4) (xy 231.14 152.4))
     (stroke (width 0) (type default))
@@
     (stroke (width 0) (type default))
   )
-  (wire (pts (xy 135.89 93.98) (xy 142.24 93.98))
+  (wire (pts (xy 135.89 88.9) (xy 142.24 88.9))
     (stroke (width 0) (type default))
   )
@@
     )
   )
-  (global_label "IR GND" (shape input) (at 142.24 93.98 0) (fields_autoplaced)
-    (effects (font (size 1.27 1.27)) (justify left))
-    (property "Intersheetrefs" "${INTERSHEET_REFS}" (at 151.9381 93.98 0)
+  (global_label "IR GND" (shape input) (at 142.24 88.9 0) (fields_autoplaced)
+    (effects (font (size 1.27 1.27)) (justify left))
+    (property "Intersheetrefs" "${INTERSHEET_REFS}" (at 151.9381 88.9 0)
       (effects (font (size 1.27 1.27)) (justify left) hide)
     )
@@
     )
   )
-  (global_label "+3.3V" (shape input) (at 142.24 99.06 0) (fields_autoplaced)
-    (effects (font (size 1.27 1.27)) (justify left))
-    (property "Intersheetrefs" "${INTERSHEET_REFS}" (at 150.91 99.06 0)
+  (global_label "+3.3V" (shape input) (at 142.24 93.98 0) (fields_autoplaced)
+    (effects (font (size 1.27 1.27)) (justify left))
+    (property "Intersheetrefs" "${INTERSHEET_REFS}" (at 150.91 93.98 0)
       (effects (font (size 1.27 1.27)) (justify left) hide)
     )
@@
     )
   )
-  (global_label "EMPTY" (shape input) (at 143.51 101.6 0) (fields_autoplaced)
-    (effects (font (size 1.27 1.27)) (justify left))
-    (property "Intersheetrefs" "${INTERSHEET_REFS}" (at 152.4218 101.6 0)
+  (global_label "EMPTY" (shape input) (at 143.51 96.52 0) (fields_autoplaced)
+    (effects (font (size 1.27 1.27)) (justify left))
+    (property "Intersheetrefs" "${INTERSHEET_REFS}" (at 152.4218 96.52 0)
       (effects (font (size 1.27 1.27)) (justify left) hide)
     )
@@
     )
   )
-  (global_label "+5V" (shape input) (at 142.24 96.52 0) (fields_autoplaced)
-    (effects (font (size 1.27 1.27)) (justify left))
-    (property "Intersheetrefs" "${INTERSHEET_REFS}" (at 149.0957 96.52 0)
+  (global_label "+5V" (shape input) (at 142.24 91.44 0) (fields_autoplaced)
+    (effects (font (size 1.27 1.27)) (justify left))
+    (property "Intersheetrefs" "${INTERSHEET_REFS}" (at 149.0957 91.44 0)
       (effects (font (size 1.27 1.27)) (justify left) hide)
     )
@@
     )
   )
-  (symbol (lib_id "Device:R") (at 139.7 101.6 270) (mirror x) (unit 1)
-    (in_bom yes) (on_board yes) (dnp no)
-    (property "Reference" "R17" (at 139.7 104.14 90)
-      (effects (font (size 1.27 1.27)))
-    )
-    (property "Value" "10K" (at 139.7 101.6 90)
-      (effects (font (size 1.27 1.27)))
-    )
-    (property "Footprint" "Resistor_THT:R_Axial_DIN0207_L6.3mm_D2.5mm_P2.54mm_Vertical" (at 139.7 103.378 90)
-      (effects (font (size 1.27 1.27)) hide)
-    )
-    (property "Datasheet" "~" (at 139.7 101.6 0)
+  (symbol (lib_id "Device:R") (at 139.7 96.52 270) (mirror x) (unit 1)
+    (in_bom yes) (on_board yes) (dnp no)
+    (property "Reference" "R17" (at 139.7 99.06 90)
+      (effects (font (size 1.27 1.27)))
+    )
+    (property "Value" "10K" (at 139.7 96.52 90)
+      (effects (font (size 1.27 1.27)))
+    )
+    (property "Footprint" "Resistor_THT:R_Axial_DIN0207_L6.3mm_D2.5mm_P2.54mm_Vertical" (at 139.7 98.298 90)
+      (effects (font (size 1.27 1.27)) hide)
+    )
+    (property "Datasheet" "~" (at 139.7 96.52 0)
       (effects (font (size 1.27 1.27)) hide)
     )
@@
         (path "/21047f2f-d4ba-4d74-abfd-549d2dbb0ef3"
           (reference "R3") (unit 1)
+        )
+      )
+    )
+  )
+  (symbol (lib_id "power:GND") (at 143.51 101.6 90) (unit 1)
+    (in_bom yes) (on_board yes) (dnp no)
+    (property "Reference" "#PWR05" (at 149.86 101.6 0)
+      (effects (font (size 1.27 1.27)) hide)
+    )
+    (property "Value" "GND" (at 147.32 101.6 0)
+      (effects (font (size 1.27 1.27)))
+    )
+    (property "Footprint" "" (at 143.51 101.6 0)
+      (effects (font (size 1.27 1.27)) hide)
+    )
+    (property "Datasheet" "" (at 143.51 101.6 0)
+      (effects (font (size 1.27 1.27)) hide)
+    )
+    (pin "1")
+    (instances
+      (project "VMFB-MC"
+        (path "/21047f2f-d4ba-4d74-abfd-549d2dbb0ef3"
+          (reference "#PWR05") (unit 1)
         )
       )
@@
     )
   )
-  (symbol (lib_id "Connector:Conn_01x04_Pin") (at 130.81 96.52 0) (unit 1)
+  (symbol (lib_id "Connector:Conn_01x04_Pin") (at 130.81 91.44 0) (unit 1)
     (in_bom yes) (on_board yes) (dnp no) (fields_autoplaced)
-    (property "Reference" "J7" (at 131.445 88.9 0)
-      (effects (font (size 1.27 1.27)))
-    )
-    (property "Value" "EMPTY" (at 131.445 91.44 0)
-      (effects (font (size 1.27 1.27)))
-    )
-    (property "Footprint" "Connector_PinHeader_2.54mm:PinHeader_1x04_P2.54mm_Vertical" (at 130.81 96.52 0)
-      (effects (font (size 1.27 1.27)) hide)
-    )
-    (property "Datasheet" "~" (at 130.81 96.52 0)
+    (property "Reference" "J7" (at 131.445 83.82 0)
+      (effects (font (size 1.27 1.27)))
+    )
+    (property "Value" "EMPTY" (at 131.445 86.36 0)
+      (effects (font (size 1.27 1.27)))
+    )
+    (property "Footprint" "Connector_PinHeader_2.54mm:PinHeader_1x04_P2.54mm_Vertical" (at 130.81 91.44 0)
+      (effects (font (size 1.27 1.27)) hide)
+    )
+    (property "Datasheet" "~" (at 130.81 91.44 0)
       (effects (font (size 1.27 1.27)) hide)
     )
@@
         )
       )
+    )
+  )
+  (symbol (lib_id "Device:R") (at 139.7 101.6 90) (unit 1)
+    (in_bom yes) (on_board yes) (dnp no)
+    (property "Reference" "R18" (at 139.7 104.14 90)
+      (effects (font (size 1.27 1.27)))
+    )
+    (property "Value" "10K" (at 139.7 101.6 90)
+      (effects (font (size 1.27 1.27)))
+    )
+    (property "Footprint" "Resistor_THT:R_Axial_DIN0207_L6.3mm_D2.5mm_P2.54mm_Vertical" (at 139.7 103.378 90)
+      (effects (font (size 1.27 1.27)) hide)
+    )
+    (property "Datasheet" "~" (at 139.7 101.6 0)
+      (effects (font (size 1.27 1.27)) hide)
+    )
+    (pin "1")
+    (pin "2")
+    (instances
+      (project "VMFB-MC"
+        (path "/21047f2f-d4ba-4d74-abfd-549d2dbb0ef3"
+          (reference "R18") (unit 1)
+        )
+      )

Commit message: Cleaned up BOM naming
Parts:
- J1, J3, J9: value DISPENSE -> Conn_01x04_Pin
- J2, J7: value EMPTY -> Conn_01x04_Pin
- J4: value MOTOR -> Conn_01x02_Pin
- J5: value PIR -> Conn_01x03_Pin
- J8: value DEPOSIT -> Conn_01x04_Pin
- Q1, Q2, Q3, Q4, Q5, Q6, Q9: value Q_Photo_NPN -> SFH313FA-2/3
- R14, R15: value 1K -> 10K
Changed lines of the file:
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@@
       (effects (font (size 1.27 1.27)) (justify left))
     )
-    (property "Value" "Q_Photo_NPN" (at 252.73 110.49 0)
+    (property "Value" "SFH313FA-2/3" (at 252.73 110.49 0)
       (effects (font (size 1.27 1.27)) (justify left))
     )
@@
       (effects (font (size 1.27 1.27)) (justify left))
     )
-    (property "Value" "Q_Photo_NPN" (at 247.65 147.8407 0)
+    (property "Value" "SFH313FA-2/3" (at 247.65 147.8407 0)
       (effects (font (size 1.27 1.27)) (justify left))
     )
@@
       (effects (font (size 1.27 1.27)) (justify left))
     )
-    (property "Value" "Q_Photo_NPN" (at 233.68 147.8407 0)
+    (property "Value" "SFH313FA-2/3" (at 233.68 147.8407 0)
       (effects (font (size 1.27 1.27)) (justify left))
     )
@@
       (effects (font (size 1.27 1.27)))
     )
-    (property "Value" "1K" (at 88.9 101.6 90)
+    (property "Value" "10K" (at 88.9 101.6 90)
       (effects (font (size 1.27 1.27)))
     )
@@
       (effects (font (size 1.27 1.27)) (justify left))
     )
-    (property "Value" "Q_Photo_NPN" (at 219.71 147.8407 0)
+    (property "Value" "SFH313FA-2/3" (at 219.71 147.8407 0)
       (effects (font (size 1.27 1.27)) (justify left))
     )
@@
       (effects (font (size 1.27 1.27)))
     )
-    (property "Value" "EMPTY" (at 131.445 86.36 0)
+    (property "Value" "Conn_01x04_Pin" (at 131.445 86.36 0)
       (effects (font (size 1.27 1.27)))
     )
@@
       (effects (font (size 1.27 1.27)) (justify left))
     )
-    (property "Value" "Q_Photo_NPN" (at 198.12 97.0407 0)
+    (property "Value" "SFH313FA-2/3" (at 198.12 97.0407 0)
       (effects (font (size 1.27 1.27)) (justify left))
     )
@@
       (effects (font (size 1.27 1.27)) (justify left))
     )
-    (property "Value" "Q_Photo_NPN" (at 238.76 110.49 0)
+    (property "Value" "SFH313FA-2/3" (at 238.76 110.49 0)
       (effects (font (size 1.27 1.27)) (justify left))
     )
@@
       (effects (font (size 1.27 1.27)))
     )
-    (property "Value" "DEPOSIT" (at 132.715 109.22 0)
+    (property "Value" "Conn_01x04_Pin" (at 132.715 109.22 0)
       (effects (font (size 1.27 1.27)))
     )
@@
       (effects (font (size 1.27 1.27)))
     )
-    (property "Value" "PIR" (at 131.445 66.04 0)
+    (property "Value" "Conn_01x03_Pin" (at 131.445 66.04 0)
       (effects (font (size 1.27 1.27)))
     )
@@
       (effects (font (size 1.27 1.27)))
     )
-    (property "Value" "1K" (at 78.74 60.96 90)
+    (property "Value" "10K" (at 78.74 60.96 90)
       (effects (font (size 1.27 1.27)))
     )
@@
       (effects (font (size 1.27 1.27)) (justify left))
     )
-    (property "Value" "Q_Photo_NPN" (at 204.47 147.8407 0)
+    (property "Value" "SFH313FA-2/3" (at 204.47 147.8407 0)
       (effects (font (size 1.27 1.27)) (justify left))
     )
@@
       (effects (font (size 1.27 1.27)))
     )
-    (property "Value" "MOTOR" (at 131.445 44.45 0)
+    (property "Value" "Conn_01x02_Pin" (at 131.445 44.45 0)
       (effects (font (size 1.27 1.27)))
     )
@@
       (effects (font (size 1.27 1.27)))
     )
-    (property "Value" "DISPENSE" (at 225.425 90.17 0)
+    (property "Value" "Conn_01x04_Pin" (at 225.425 90.17 0)
       (effects (font (size 1.27 1.27)))
     )
@@
       (effects (font (size 1.27 1.27)))
     )
-    (property "Value" "DISPENSE" (at 182.245 134.62 0)
+    (property "Value" "Conn_01x04_Pin" (at 182.245 134.62 0)
       (effects (font (size 1.27 1.27)))
     )
@@
       (effects (font (size 1.27 1.27)))
     )
-    (property "Value" "DISPENSE" (at 133.985 127 0)
+    (property "Value" "Conn_01x04_Pin" (at 133.985 127 0)
       (effects (font (size 1.27 1.27)))
     )
@@
       (effects (font (size 1.27 1.27)))
     )
-    (property "Value" "EMPTY" (at 175.895 83.82 0)
-      (effects (font (size 1.27 1.27)))
-    )
+    (property "Value" "Conn_01x04_Pin" (at 175.895 83.82 0)
+      (effects (font (size 1.27 1.27)))
+    )

Commit message: clean up
removed some unnecessary components and revised component placement.
Parts:
- removed R10, R11, R16, R17: 10K, Resistor_THT:R_Axial_DIN0207_L6.3mm_D2.5mm_P2.54mm_Vertical, symbol Device:R
- renumbered J6 to J10, J7 to J6, J8 to J7, J9 to J8, J10 to J9, R12 to R10, R13 to R11, R14 to R12, R15 to R13, R18 to R14
Connections:
- net DEPOSIT SIG: now also R8.2, U1.5 (+)
- net DISPENSE: now also R11.2; no longer R11.1
- net DISPENSE SIG: now also R9.2, U1.3 (+)
- net EMPTY: now also J6.4 (Pin_4), R14.1
- net GND: now also R9.1; no longer R9.2
- net PIR: now also J5.3 (Pin_3)
- net at U1.1: now also R11.1; no longer R11.2
Other:
- moved on the sheet: R11
